Commit message: RMF fleet adapter nav2 for Ionic demo (#8)
* Add basic dispenser pick and place

Signed-off-by: Luca Della Vedova <lucadv@intrinsic.ai>

* Add rmf message to dependencies

Signed-off-by: Luca Della Vedova <lucadv@intrinsic.ai>

* Update branches / dependencies

Signed-off-by: Luca Della Vedova <lucadv@intrinsic.ai>

* Add nav2 and custom branch

Signed-off-by: Luca Della Vedova <lucadv@intrinsic.ai>

* Fix rviz and nav2 demo

Signed-off-by: Luca Della Vedova <lucadv@intrinsic.ai>

* Fleet adapter nav2 for Ionic demo (#5)

* Add fleet adapter template

Signed-off-by: Xiyu Oh <xiyu@openrobotics.org>

* Ac/tf listener (#1)

* Basic TF listener, not tested yet

Signed-off-by: Aaron Chong <aaronchongth@gmail.com>

* Started README

Signed-off-by: Aaron Chong <aaronchongth@gmail.com>

---------

Signed-off-by: Aaron Chong <aaronchongth@gmail.com>

* Fleet adapter bringup (#3)

* Working adapter but wrong tf read

Signed-off-by: Xiyu Oh <xiyu@openrobotics.org>

* Fix reference coordinates, tfs,typo (#4)

Signed-off-by: Aaron Chong <aaronchongth@gmail.com>

* Working fleet adapter with demo map

Signed-off-by: Xiyu Oh <xiyu@openrobotics.org>

---------

Signed-off-by: Xiyu Oh <xiyu@openrobotics.org>
Signed-off-by: Aaron Chong <aaronchongth@gmail.com>
Co-authored-by: Aaron Chong <aaronchongth@gmail.com>

* Works with gazebosim/ionic_demo#1

Signed-off-by: Aaron Chong <aaronchongth@gmail.com>

* Update instructions

Signed-off-by: Aaron Chong <aaronchongth@gmail.com>

* Ros package and nav2 demo (#1)

* launching the demo world
* Added new laser scan and updated launch file
* Setting up ionic_demo as its own pacakge
* Updated with gif
* Clean up and add license
* Remove unused launch file
* Add media

---------

Signed-off-by: Aaron Chong <aaronchongth@gmail.com>
Co-authored-by: Tully Foote <tullyfoote@intrinsic.ai>

* Add docker file and workflow to publish docker images (#3)

Signed-off-by: Addisu Z. Taddese <addisu@openrobotics.org>

* Use composition for ros_gz and Gazebo in Nav2 launch files (#4)

* Reimplements the turtlebot4 launch file from nav2_bringup in order to
use composition for ros_gz and Gazebo. Hopefully, some of this will be
upstreamed to Nav2.

* This also updates the step size to 0.004 to speed up simulation

Signed-off-by: Addisu Z. Taddese <addisu@openrobotics.org>

* Add a tray to the turtlebot4 (#6)

* Use composition for ros_gz and Gazebo in Nav2 launch files

* Reimplements the turtlebot4 launch file from nav2_bringup in order to
use composition for ros_gz and Gazebo. Hopefully, some of this will be
upstreamed to Nav2.

* This also updates the step size to 0.004 to speed up simulation

Signed-off-by: Addisu Z. Taddese <addisu@openrobotics.org>

* Add a tray to the turtlebot4

Signed-off-by: Addisu Z. Taddese <addisu@openrobotics.org>

---------

Signed-off-by: Addisu Z. Taddese <addisu@openrobotics.org>

---------

Signed-off-by: Xiyu Oh <xiyu@openrobotics.org>
Signed-off-by: Aaron Chong <aaronchongth@gmail.com>
Signed-off-by: Addisu Z. Taddese <addisu@openrobotics.org>
Co-authored-by: Xiyu Oh <xiyu@openrobotics.org>
Co-authored-by: Xiyu <ohxiyu@gmail.com>
Co-authored-by: Tully Foote <tullyfoote@intrinsic.ai>
Co-authored-by: Addisu Z. Taddese <addisu@openrobotics.org>

* Add adapter to launch file

Signed-off-by: Xiyu Oh <xiyu@openrobotics.org>

* Fix launch file and add exec depends

Signed-off-by: Aaron Chong <aaronchongth@gmail.com>

* Add rest of dispenser logic, fix fleet adapter

Signed-off-by: Luca Della Vedova <lucadv@intrinsic.ai>

* Fix dispensor result / stage logic

Signed-off-by: Luca Della Vedova <lucadv@intrinsic.ai>

* Build docker image with RMF as well

Signed-off-by: Aaron Chong <aaronchongth@gmail.com>

* Spawn teleport ingestor model

Signed-off-by: Luca Della Vedova <lucadv@intrinsic.ai>

* Change branch of ionic_demo

Signed-off-by: Aaron Chong <aaronchongth@gmail.com>

* Add RMF to moveit launch

Signed-off-by: Luca Della Vedova <lucadv@intrinsic.ai>

* Target rmf.repos that allow skipping qt building plugins

Signed-off-by: Aaron Chong <aaronchongth@gmail.com>

* Fix dependencies

Signed-off-by: Luca Della Vedova <lucadellavr@gmail.com>

* Use correct flag to skip qt moc plugin builds

Signed-off-by: Aaron Chong <aaronchongth@gmail.com>

* Revert to use rmf_simulation main, remove cmake flag (#7)

* Revert to use rmf_simulation main, remove cmake flag

Signed-off-by: Aaron Chong <aaronchongth@gmail.com>

* Remove wget and vcs step for rmf.repos

Signed-off-by: Aaron Chong <aaronchongth@gmail.com>

---------

Signed-off-by: Aaron Chong <aaronchongth@gmail.com>

* Fix coordinates / names for delivery demo

Signed-off-by: Luca Della Vedova <lucadellavr@gmail.com>

* Remove detachable joint and use normal gripping

Signed-off-by: Luca Della Vedova <lucadellavr@gmail.com>

* Split launch files for single demos

Signed-off-by: Luca Della Vedova <lucadellavr@gmail.com>

* Tune map, nav2 inflation layer, gripper close values, added dashboard… (#8)

* Tune map, nav2 inflation layer, gripper close values, added dashboard build

Signed-off-by: Aaron Chong <aaronchongth@gmail.com>

* Attempt to build dashboard image first

Signed-off-by: Aaron Chong <aaronchongth@gmail.com>

* Add media, update readme, revert changes to workflow

Signed-off-by: Aaron Chong <aaronchongth@gmail.com>

* One liner for dashboard url

Signed-off-by: Xiyu Oh <xiyu@openrobotics.org>

* Move environment variables to moveit launch

Signed-off-by: Luca Della Vedova <lucadellavr@gmail.com>

* Build dashboard with better robot zoom values, increase yaw tolerance for nav2 to prevent wobble

Signed-off-by: Aaron Chong <aaronchongth@gmail.com>

* Increase yaw tolerance even more, revert workflow

Signed-off-by: Aaron Chong <aaronchongth@gmail.com>

* Add gitignore

Signed-off-by: Aaron Chong <aaronchongth@gmail.com>

---------

Signed-off-by: Aaron Chong <aaronchongth@gmail.com>
Signed-off-by: Xiyu Oh <xiyu@openrobotics.org>
Signed-off-by: Luca Della Vedova <lucadellavr@gmail.com>
Co-authored-by: Xiyu Oh <xiyu@openrobotics.org>
Co-authored-by: Luca Della Vedova <lucadellavr@gmail.com>

* Update dashboard docker image URL

Signed-off-by: Aaron Chong <aaronchongth@gmail.com>

---------

Signed-off-by: Luca Della Vedova <lucadv@intrinsic.ai>
Signed-off-by: Xiyu Oh <xiyu@openrobotics.org>
Signed-off-by: Aaron Chong <aaronchongth@gmail.com>
Signed-off-by: Addisu Z. Taddese <addisu@openrobotics.org>
Signed-off-by: Luca Della Vedova <lucadellavr@gmail.com>
Co-authored-by: Luca Della Vedova <lucadv@intrinsic.ai>
Co-authored-by: Aaron Chong <aaronchongth@gmail.com>
Co-authored-by: Tully Foote <tullyfoote@intrinsic.ai>
Co-authored-by: Addisu Z. Taddese <addisu@openrobotics.org>
Co-authored-by: Luca Della Vedova <lucadellavr@gmail.com>

File: ionic_demo/models/ionic_tb4.urdf.xacro (robot description, xacro)
@@ -5,5 +5,5 @@
     <parent link="tower_sensor_plate"/>
     <child link="tray"/>
-    <origin xyz="0 0 0.5"/>
+    <origin xyz="0.03 0 0.5"/>
   </joint>
   <link name="tray">
